File: pcb/gpib_adapter.sch (KiCad schematic (older format))
At the start: 27 parts, among them IC1 ATMEGA16U4, P1 ISP, P2 USB, P3 GPIO, P4 UART, P5 GPIB, P6 PWR_JMP, U1 SN75160, U2 SN75161

Commit message: Routed one more GPIO pin, changed GPIO connector
Parts:
- removed P3: GPIO, symbol CONN_5
- added P3: GPIO, symbol CONN_3X2
Connections:
- net GND: now also P3.6
- net GPIO1: now also P3.1
- net GPIO2: now also P3.2
- net GPIO3: now also P3.3
- net GPIO4: now also P3.4
- net GPIO5: now reaches IC1.37 ((ADC6/TDO)PF6)
- net GPIO5: now also P3.5
Changed lines of the file:
@@
-EESchema Schematic File Version 2  date Mon 16 Jul 2012 03:40:06 PM EEST
+EESchema Schematic File Version 2  date Mon 16 Jul 2012 04:53:42 PM EEST
 LIBS:power
 LIBS:device
@@
 DIO1
 $Comp
-L CONN_5 P3
-U 1 1 4FFF0CDC
-P 9900 4050
-F 0 "P3" V 9850 4050 50  0000 C CNN
-F 1 "GPIO" V 9950 4050 50  0000 C CNN
-	1    9900 4050
-	1    0    0    -1
-$EndComp
-$Comp
-L GND #PWR05
-U 1 1 4FFF116C
-P 9500 4300
-F 0 "#PWR05" H 9500 4300 30  0001 C CNN
-F 1 "GND" H 9500 4230 30  0001 C CNN
-	1    9500 4300
-	1    0    0    -1
-$EndComp
-$Comp
 L CONN_5 P2
 U 1 1 4FFF132F
@@
 $EndComp
 $Comp
-L GND #PWR06
+L GND #PWR05
 U 1 1 500128DE
 P 6600 2000
-F 0 "#PWR06" H 6600 2000 30  0001 C CNN
+F 0 "#PWR05" H 6600 2000 30  0001 C CNN
 F 1 "GND" H 6600 1930 30  0001 C CNN
 	1    6600 2000
@@
 $EndComp
 $Comp
-L +5V #PWR07
+L +5V #PWR06
 U 1 1 500128E4
 P 6600 1500
-F 0 "#PWR07" H 6600 1590 20  0001 C CNN
+F 0 "#PWR06" H 6600 1590 20  0001 C CNN
 F 1 "+5V" H 6600 1590 30  0000 C CNN
 	1    6600 1500
@@
 $EndComp
 $Comp
-L GND #PWR08
+L GND #PWR07
 U 1 1 50012A5D
 P 6900 3800
-F 0 "#PWR08" H 6900 3800 30  0001 C CNN
+F 0 "#PWR07" H 6900 3800 30  0001 C CNN
 F 1 "GND" H 6900 3730 30  0001 C CNN
 	1    6900 3800
@@
 $EndComp
 $Comp
-L GND #PWR09
+L GND #PWR08
 U 1 1 50012AED
 P 6600 4350
-F 0 "#PWR09" H 6600 4350 30  0001 C CNN
+F 0 "#PWR08" H 6600 4350 30  0001 C CNN
 F 1 "GND" H 6600 4280 30  0001 C CNN
 	1    6600 4350
@@
 $EndComp
 $Comp
-L +5V #PWR010
+L +5V #PWR09
 U 1 1 50012B6E
 P 6600 3850
-F 0 "#PWR010" H 6600 3940 20  0001 C CNN
+F 0 "#PWR09" H 6600 3940 20  0001 C CNN
 F 1 "+5V" H 6600 3940 30  0000 C CNN
 	1    6600 3850
@@
 $EndComp
 $Comp
-L GND #PWR011
+L GND #PWR010
 U 1 1 50012C6D
 P 6900 6100
-F 0 "#PWR011" H 6900 6100 30  0001 C CNN
+F 0 "#PWR010" H 6900 6100 30  0001 C CNN
 F 1 "GND" H 6900 6030 30  0001 C CNN
 	1    6900 6100
@@
 $EndComp
 $Comp
-L +5V #PWR012
+L +5V #PWR011
 U 1 1 500131BC
 P 5700 3350
-F 0 "#PWR012" H 5700 3440 20  0001 C CNN
+F 0 "#PWR011" H 5700 3440 20  0001 C CNN
 F 1 "+5V" H 5700 3440 30  0000 C CNN
 	1    5700 3350
@@
 $EndComp
 $Comp
-L GND #PWR013
+L GND #PWR012
 U 1 1 50017B22
 P 1700 3450
-F 0 "#PWR013" H 1700 3450 30  0001 C CNN
+F 0 "#PWR012" H 1700 3450 30  0001 C CNN
 F 1 "GND" H 1700 3380 30  0001 C CNN
 	1    1700 3450
@@
 $EndComp
 $Comp
-L GND #PWR014
+L GND #PWR013
 U 1 1 50017BBF
 P 2800 4050
-F 0 "#PWR014" H 2800 4050 30  0001 C CNN
+F 0 "#PWR013" H 2800 4050 30  0001 C CNN
 F 1 "GND" H 2800 3980 30  0001 C CNN
 	1    2800 4050
@@
 Text Label 5150 5050 0    60   ~ 0
 GPIO4
-Text Label 9200 3850 0    60   ~ 0
+Text Label 9200 4000 0    60   ~ 0
 GPIO1
-Text Label 9200 3950 0    60   ~ 0
+Text Label 10350 4000 0    60   ~ 0
 GPIO2
-Text Label 9200 4050 0    60   ~ 0
+Text Label 9200 4100 0    60   ~ 0
 GPIO3
-Text Label 9200 4150 0    60   ~ 0
+Text Label 10350 4100 0    60   ~ 0
 GPIO4
 Text Label 7550 2300 0    60   ~ 0
@@
 $EndComp
 $Comp
-L GND #PWR015
+L GND #PWR014
 U 1 1 5001D786
 P 9550 4900
-F 0 "#PWR015" H 9550 4900 30  0001 C CNN
+F 0 "#PWR014" H 9550 4900 30  0001 C CNN
 F 1 "GND" H 9550 4830 30  0001 C CNN
 	1    9550 4900
@@
 TXD
 $Comp
-L +5V #PWR016
+L +5V #PWR015
 U 1 1 5001DC92
 P 9200 5050
-F 0 "#PWR016" H 9200 5140 20  0001 C CNN
+F 0 "#PWR015" H 9200 5140 20  0001 C CNN
 F 1 "+5V" H 9200 5140 30  0000 C CNN
 	1    9200 5050
@@
 $EndComp
 $Comp
-L VCC #PWR017
+L VCC #PWR016
 U 1 1 5001DDF8
 P 2300 2750
-F 0 "#PWR017" H 2300 2850 30  0001 C CNN
+F 0 "#PWR016" H 2300 2850 30  0001 C CNN
 F 1 "VCC" H 2300 2850 30  0000 C CNN
 	1    2300 2750
@@
 $EndComp
 $Comp
-L VCC #PWR018
+L VCC #PWR017
 U 1 1 5001DFEA
 P 9450 5100
-F 0 "#PWR018" H 9450 5200 30  0001 C CNN
+F 0 "#PWR017" H 9450 5200 30  0001 C CNN
 F 1 "VCC" H 9450 5200 30  0000 C CNN
 	1    9450 5100
@@
 $EndComp
 $Comp
-L GND #PWR019
+L GND #PWR018
 U 1 1 5001E0AA
 P 9550 5450
-F 0 "#PWR019" H 9550 5450 30  0001 C CNN
+F 0 "#PWR018" H 9550 5450 30  0001 C CNN
 F 1 "GND" H 9550 5380 30  0001 C CNN
 	1    9550 5450
@@
 $EndComp
 $Comp
-L VDD #PWR020
+L VDD #PWR019
 U 1 1 5001E15D
 P 9450 4750
-F 0 "#PWR020" H 9450 4850 30  0001 C CNN
+F 0 "#PWR019" H 9450 4850 30  0001 C CNN
 F 1 "VDD" H 9450 4860 30  0000 C CNN
 	1    9450 4750
@@
 $EndComp
 $Comp
-L VDD #PWR021
+L VDD #PWR020
 U 1 1 5001E174
 P 9450 5300
-F 0 "#PWR021" H 9450 5400 30  0001 C CNN
+F 0 "#PWR020" H 9450 5400 30  0001 C CNN
 F 1 "VDD" H 9450 5410 30  0000 C CNN
 	1    9450 5300
@@
 	5100 5250 5150 5250
 Wire Wire Line
-	9500 4300 9500 4250
-Wire Wire Line
 	5100 4750 5150 4750
 Wire Wire Line
@@
 	5100 5050 5150 5050
 Wire Wire Line
-	9200 3850 9500 3850
-Wire Wire Line
-	9200 3950 9500 3950
-Wire Wire Line
-	9200 4050 9500 4050
-Wire Wire Line
-	9200 4150 9500 4150
+	9200 4000 9500 4000
+Wire Wire Line
+	9200 4100 9500 4100
+Wire Wire Line
+	9200 4200 9500 4200
 Wire Wire Line
 	7500 2300 7900 2300
@@
 $EndComp
 $Comp
-L GND #PWR022
+L GND #PWR021
 U 1 1 5002765A
 P 10300 5950
-F 0 "#PWR022" H 10300 5950 30  0001 C CNN
+F 0 "#PWR021" H 10300 5950 30  0001 C CNN
 F 1 "GND" H 10300 5880 30  0001 C CNN
 	1    10300 5950
@@
 $EndComp
 $Comp
-L +5V #PWR023
+L +5V #PWR022
 U 1 1 50027660
 P 10300 5650
-F 0 "#PWR023" H 10300 5740 20  0001 C CNN
+F 0 "#PWR022" H 10300 5740 20  0001 C CNN
 F 1 "+5V" H 10300 5740 30  0000 C CNN
 	1    10300 5650
@@
 $EndComp
 $Comp
-L GND #PWR024
+L GND #PWR023
 U 1 1 50027FCC
 P 8250 5350
-F 0 "#PWR024" H 8250 5350 30  0001 C CNN
+F 0 "#PWR023" H 8250 5350 30  0001 C CNN
 F 1 "GND" H 8250 5280 30  0001 C CNN
 	1    8250 5350
@@
 	2750 2300 2900 2300
 Wire Wire Line
-	3700 1650 2050 1650
+	2050 1650 3700 1650
 Wire Wire Line
 	2050 1650 2050 2300
@@
 Wire Bus Line
 	8000 2200 10800 2200
+$Comp
+L GND #PWR024
+U 1 1 5004181A
+P 10300 4250
+F 0 "#PWR024" H 10300 4250 30  0001 C CNN
+F 1 "GND" H 10300 4180 30  0001 C CNN
+	1    10300 4250
+	1    0    0    -1
+$EndComp
+Text Label 9200 4200 0    60   ~ 0
+GPIO5
+$Comp
+L CONN_3X2 P3
+U 1 1 50041A7E
+P 9900 4150
+F 0 "P3" H 9900 4400 50  0000 C CNN
+F 1 "GPIO" V 9900 4200 40  0000 C CNN
+	1    9900 4150
+	1    0    0    -1
+$EndComp
+Wire Wire Line
+	10300 4250 10300 4200
+Wire Wire Line
+	10300 4000 10350 4000
+Wire Wire Line
+	10300 4100 10350 4100
+Text Label 5150 5150 0    60   ~ 0
+GPIO5
+Wire Wire Line
+	5150 5150 5100 5150
 $EndSCHEMATC
